Commit message: Gazebo

File: diff_drive/urdf/ddrive.gazebo.xacro (robot description, xacro)
@@ -10,5 +10,5 @@
 <xacro:property name="R2" value="${ddrive['R2']}" />
 <xacro:property name="L2" value="${ddrive['L2']}" />
-<gazebo reference="base_link">
+<gazebo reference="body">
   <material>Gazebo/Blue</material>
 </gazebo>

File: diff_drive/urdf/ddrive.urdf.xacro (robot description, xacro)
@@ -14,5 +14,12 @@
 <xacro:property name="m_wheel" value="0.4" />
 <xacro:property name="m_caster" value="0.4" />
-<link name="base_link" >
+<link name="base_link"/>
+<joint name="dummy" type = "fixed">
+  <origin xyz="0 0 0" rpy="0 0 0" />
+  <parent link="base_link" />
+  <child link="body" />
+</joint>
+<link name="body" >
+  <origin xyz="0 0 0" rpy="0 0 0" />
   <visual>
     <geometry>
@@ -43,5 +50,5 @@
   <origin xyz="${L/2} ${W/2 + L1/2} 0" rpy="${-pi/2} 0 0" />
   <axis xyz =" 0 0 1"/>
-  <parent link="base_link" />
+  <parent link="body" />
   <child link="left_wheel" />
 </joint>
@@ -75,5 +82,5 @@
   <origin xyz="${L/2} ${-W/2 - L1/2} 0" rpy="${-pi/2} 0 0" />
   <axis xyz =" 0 0 1"/>
-  <parent link="base_link" />
+  <parent link="body" />
   <child link="right_wheel" />
 </joint>
@@ -107,5 +114,5 @@
   <origin xyz="${-L/2 + R2/2} 0 ${H/2 + R2}" rpy="${-pi/2} 0 0" />
   <axis xyz =" 0 0 1"/>
-  <parent link="base_link" />
+  <parent link="body" />
   <child link="top_caster" />
 </joint>
@@ -139,5 +146,5 @@
   <origin xyz="${-L/2 + R2/2} 0 ${-H/2 - R2}" rpy="${-pi/2} 0 0" />
   <axis xyz =" 0 0 1"/>
-  <parent link="base_link" />
+  <parent link="body" />
   <child link="bottom_caster" />
 </joint>

Commit message: diff_drive works

File: diff_drive/urdf/ddrive.gazebo.xacro (robot description, xacro)
@@ -14,5 +14,5 @@
 </gazebo>
 <gazebo reference="left_wheel">
-  <material>Gazebo/Green</material>
+  <material>Gazebo/Wood</material>
   <mu1>999</mu1>
   <mu2>999</mu2>
@@ -24,5 +24,5 @@
 </gazebo>
 <gazebo reference="right_wheel">
-  <material>Gazebo/Green</material>
+  <material>Gazebo/Wood</material>
   <mu1>999</mu1>
   <mu2>999</mu2>
@@ -54,24 +54,24 @@
 </gazebo>
 <gazebo>
-<plugin name="differential_drive_controller" filename="libgazebo_ros_diff_drive.so">
-<rosDebugLevel>na</rosDebugLevel>
-<alwaysOn>true</alwaysOn>
-<updateRate>100</updateRate>
-<leftJoint>right_wheel</leftJoint>
-<rightJoint>left_wheel</rightJoint>
-<wheelSeparation>${W+L1}</wheelSeparation>
-<wheelDiameter>${R1}</wheelDiameter>
-<wheelTorque>20</wheelTorque>
-<commandTopic>diff/cmd_vel</commandTopic>
-<odometryTopic>diff/odom</odometryTopic>
-<odometryFrame>odom</odometryFrame>
-<robotBaseFrame>base_link</robotBaseFrame>
-<publishWheelTF>false</publishWheelTF>
-<publishOdomTF>true</publishOdomTF>
-<publishWheelJointState>true</publishWheelJointState>
-<wheelAcceleration>false</wheelAcceleration>
-<odometrySource>world</odometrySource>
-<publishTf>1</publishTf>
-</plugin>
+  <plugin name="differential_drive_controller" filename="libgazebo_ros_diff_drive.so">
+  <rosDebugLevel>na</rosDebugLevel>
+  <alwaysOn>true</alwaysOn>
+  <updateRate>100</updateRate>
+  <leftJoint>right_wheel_joint</leftJoint>
+  <rightJoint>left_wheel_joint</rightJoint>
+  <wheelSeparation>${W+L1}</wheelSeparation>
+  <wheelDiameter>${R1*2}</wheelDiameter>
+  <wheelTorque>20</wheelTorque>
+  <commandTopic>diff/cmd_vel</commandTopic>
+  <odometryTopic>diff/odom</odometryTopic>
+  <odometryFrame>odom</odometryFrame>
+  <robotBaseFrame>base_link</robotBaseFrame>
+  <publishWheelTF>false</publishWheelTF>
+  <publishOdomTF>true</publishOdomTF>
+  <publishWheelJointState>true</publishWheelJointState>
+  <wheelAcceleration>false</wheelAcceleration>
+  <odometrySource>world</odometrySource>
+  <publishTf>1</publishTf>
+  </plugin>
 </gazebo>
 </robot>
